File: Kicad/MVS Pause Button.kicad_pcb (KiCad board)
At the start: 2 copper layers, 18.4 x 12 mm, 15 parts, among them J1 Conn_01x01_Male, J2 Conn_01x01_Male, J3 Conn_01x01_Male, J4 Conn_01x01_Male

Commit message: v1.1
v1.1
Parts:
- added R3: 10k, Resistor_SMD:R_0603_1608Metric_Pad0.98x0.95mm_HandSolder, F.Cu at (114.3, 44.7)
- REF** (x3): moved to F.Cu
- moved REF** 16.7 mm to (122.8, 46.0), turned to 0 degrees
- moved C1 5.82 mm to (119.2, 46.0)
- moved POR1 0.40 mm to (113.8, 48.2)
- moved REF** 0.28 mm to (106.0, 53.5), turned to 0 degrees
- moved C2 0.27 mm to (113.8, 51.8)
- moved REF** 0.22 mm to (115.1, 53.5), turned to 0 degrees
- renumbered DC1 to C2, R2 to R1, R1 to R2
Connections:
- FLP1 pad 3: DIP8 -> Net-(FLP1-Pad3)
- INV1 pad 4: DIP8 -> Net-(FLP1-Pad3)
Routing:
- net DIP8: track 15.5 -> 2.62 mm, vias 1 -> 0
- net Net-(FLP1-Pad3): track 0.00 -> 9.02 mm
- net INV_In: track 6.85 -> 13.6 mm, vias 0 -> 3
- net GND: track 6.78 -> 4.44 mm, vias 3 -> 4
Other:
- board text added: "C1"
- board text added: "C2"
- board text removed: "100nF"
