File: Kicad/MVS Pause Button.kicad_sch (KiCad schematic)
At the start: 11 parts, among them J1 Conn_01x01_Male, J2 Conn_01x01_Male, J3 Conn_01x01_Male, J4 Conn_01x01_Male

Commit message: v1.1
v1.1
Parts:
- added R3: 10k, Resistor_SMD:R_0603_1608Metric_Pad0.98x0.95mm_HandSolder, symbol Device:R
- renumbered DC1 to C2, R2 to R1, R1 to R2
Connections:
- net DIP8: now also R3.1; no longer FLP1.3 (D), INV1.4 (2Y)
- new net: FLP1.3 (D), INV1.4 (2Y), R3.2
Other:
- moved on the sheet: C2
Changed lines of the file:
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@@
-    (stroke (width 0) (type default) (color 0 0 0 0))
-  )
-  (wire (pts (xy 135.89 83.82) (xy 134.62 83.82))
     (stroke (width 0) (type default) (color 0 0 0 0))
   )
@@
     (stroke (width 0) (type default) (color 0 0 0 0))
   )
-  (wire (pts (xy 134.62 83.82) (xy 134.62 81.28))
+  (wire (pts (xy 134.62 81.28) (xy 134.62 91.44))
     (stroke (width 0) (type default) (color 0 0 0 0))
   )
@@
     )
   )
-  (global_label "DIP8" (shape input) (at 135.89 83.82 0) (fields_autoplaced)
+  (global_label "DIP8" (shape input) (at 142.24 91.44 0) (fields_autoplaced)
     (effects (font (size 1.27 1.27)) (justify left))
-    (property "Intersheet References" "${INTERSHEET_REFS}" (id 0) (at 142.6574 83.7406 0)
+    (property "Intersheet References" "${INTERSHEET_REFS}" (id 0) (at 149.0074 91.3606 0)
       (effects (font (size 1.27 1.27)) (justify left) hide)
     )
   )
-  (symbol (lib_id "power:+5V") (at 134.62 93.98 90) (unit 1)
-    (in_bom yes) (on_board yes)
-    (property "Reference" "#PWR0114" (id 0) (at 138.43 93.98 0)
-      (effects (font (size 1.27 1.27)) hide)
-    )
-    (property "Value" "+5V" (id 1) (at 132.08 93.98 90)
+  (symbol (lib_id "power:+5V") (at 100.33 93.98 90) (unit 1)
+    (in_bom yes) (on_board yes)
+    (property "Reference" "#PWR0114" (id 0) (at 104.14 93.98 0)
+      (effects (font (size 1.27 1.27)) hide)
+    )
+    (property "Value" "+5V" (id 1) (at 97.79 93.98 90)
       (effects (font (size 1.27 1.27)) (justify left))
     )
-    (property "Footprint" "" (id 2) (at 134.62 93.98 0)
-      (effects (font (size 1.27 1.27)) hide)
-    )
-    (property "Datasheet" "" (id 3) (at 134.62 93.98 0)
+    (property "Footprint" "" (id 2) (at 100.33 93.98 0)
+      (effects (font (size 1.27 1.27)) hide)
+    )
+    (property "Datasheet" "" (id 3) (at 100.33 93.98 0)
       (effects (font (size 1.27 1.27)) hide)
     )
@@
   (symbol (lib_id "Device:R") (at 90.17 77.47 180) (unit 1)
     (in_bom yes) (on_board yes)
-    (property "Reference" "R1" (id 0) (at 90.17 77.47 90))
+    (property "Reference" "R2" (id 0) (at 90.17 77.47 90))
     (property "Value" "10k" (id 1) (at 92.71 77.47 90))
     (property "Footprint" "Resistor_SMD:R_0603_1608Metric_Pad0.98x0.95mm_HandSolder" (id 2) (at 91.948 77.47 90)
@@
     (pin "3")
   )
-  (symbol (lib_id "power:GND") (at 142.24 93.98 90) (unit 1)
-    (in_bom yes) (on_board yes) (fields_autoplaced)
-    (property "Reference" "#PWR0112" (id 0) (at 148.59 93.98 0)
-      (effects (font (size 1.27 1.27)) hide)
-    )
-    (property "Value" "GND" (id 1) (at 146.05 93.9799 90)
-      (effects (font (size 1.27 1.27)) (justify right))
-    )
-    (property "Footprint" "" (id 2) (at 142.24 93.98 0)
-      (effects (font (size 1.27 1.27)) hide)
-    )
-    (property "Datasheet" "" (id 3) (at 142.24 93.98 0)
+  (symbol (lib_id "power:GND") (at 107.95 93.98 90) (unit 1)
+    (in_bom yes) (on_board yes) (fields_autoplaced)
+    (property "Reference" "#PWR0112" (id 0) (at 114.3 93.98 0)
+      (effects (font (size 1.27 1.27)) hide)
+    )
+    (property "Value" "GND" (id 1) (at 111.76 93.9799 90)
+      (effects (font (size 1.27 1.27)) (justify right))
+    )
+    (property "Footprint" "" (id 2) (at 107.95 93.98 0)
+      (effects (font (size 1.27 1.27)) hide)
+    )
+    (property "Datasheet" "" (id 3) (at 107.95 93.98 0)
       (effects (font (size 1.27 1.27)) hide)
     )
@@
     )
     (pin "1")
+  )
+  (symbol (lib_id "Device:R") (at 138.43 91.44 270) (unit 1)
+    (in_bom yes) (on_board yes)
+    (property "Reference" "R3" (id 0) (at 138.43 91.44 90))
+    (property "Value" "10k" (id 1) (at 138.43 88.9 90))
+    (property "Footprint" "Resistor_SMD:R_0603_1608Metric_Pad0.98x0.95mm_HandSolder" (id 2) (at 138.43 89.662 90)
+      (effects (font (size 1.27 1.27)) hide)
+    )
+    (property "Datasheet" "~" (id 3) (at 138.43 91.44 0)
+      (effects (font (size 1.27 1.27)) hide)
+    )
+    (pin "1")
+    (pin "2")
   )
   (symbol (lib_id "power:+5V") (at 177.8 77.47 180) (unit 1)
@@
     (pin "1")
   )
-  (symbol (lib_id "Device:C") (at 138.43 93.98 90) (unit 1)
-    (in_bom yes) (on_board yes)
-    (property "Reference" "DC1" (id 0) (at 134.62 91.44 90))
-    (property "Value" "100nF" (id 1) (at 143.51 91.44 90))
-    (property "Footprint" "Capacitor_SMD:C_0603_1608Metric_Pad1.08x0.95mm_HandSolder" (id 2) (at 142.24 93.0148 0)
-      (effects (font (size 1.27 1.27)) hide)
-    )
-    (property "Datasheet" "~" (id 3) (at 138.43 93.98 0)
+  (symbol (lib_id "Device:C") (at 104.14 93.98 90) (unit 1)
+    (in_bom yes) (on_board yes)
+    (property "Reference" "C2" (id 0) (at 100.33 91.44 90))
+    (property "Value" "100nF" (id 1) (at 109.22 91.44 90))
+    (property "Footprint" "Capacitor_SMD:C_0603_1608Metric_Pad1.08x0.95mm_HandSolder" (id 2) (at 107.95 93.0148 0)
+      (effects (font (size 1.27 1.27)) hide)
+    )
+    (property "Datasheet" "~" (id 3) (at 104.14 93.98 0)
       (effects (font (size 1.27 1.27)) hide)
     )
@@
   (symbol (lib_id "Device:R") (at 96.52 73.66 90) (unit 1)
     (in_bom yes) (on_board yes)
-    (property "Reference" "R2" (id 0) (at 96.52 73.66 90))
+    (property "Reference" "R1" (id 0) (at 96.52 73.66 90))
     (property "Value" "1k" (id 1) (at 96.52 76.2 90))
     (property "Footprint" "Resistor_SMD:R_0603_1608Metric_Pad0.98x0.95mm_HandSolder" (id 2) (at 96.52 75.438 90)
@@
     )
     (path "/7baf9ce9-d47b-49d6-9176-8b6929776299"
-      (reference "DC1") (unit 1) (value "100nF") (footprint "Capacitor_SMD:C_0603_1608Metric_Pad1.08x0.95mm_HandSolder")
+      (reference "C2") (unit 1) (value "100nF") (footprint "Capacitor_SMD:C_0603_1608Metric_Pad1.08x0.95mm_HandSolder")
     )
     (path "/f2de39ad-3a34-4e0d-8c37-6f00e6f07643"
@@
       (reference "POR1") (unit 1) (value "MCP100-315D") (footprint "Package_TO_SOT_SMD:SOT-23_Handsoldering")
     )
+    (path "/ec5c25f0-3fe8-427a-aa7d-58556619d526"
+      (reference "R1") (unit 1) (value "1k") (footprint "Resistor_SMD:R_0603_1608Metric_Pad0.98x0.95mm_HandSolder")
+    )
     (path "/232e5e62-2711-4d61-9e04-320a298250b9"
-      (reference "R1") (unit 1) (value "10k") (footprint "Resistor_SMD:R_0603_1608Metric_Pad0.98x0.95mm_HandSolder")
-    )
-    (path "/ec5c25f0-3fe8-427a-aa7d-58556619d526"
-      (reference "R2") (unit 1) (value "1k") (footprint "Resistor_SMD:R_0603_1608Metric_Pad0.98x0.95mm_HandSolder")
-    )
-  )
+      (reference "R2") (unit 1) (value "10k") (footprint "Resistor_SMD:R_0603_1608Metric_Pad0.98x0.95mm_HandSolder")
+    )
+    (path "/6c5fe62b-2a83-4a65-b6bc-95eae718d02c"
+      (reference "R3") (unit 1) (value "10k") (footprint "Resistor_SMD:R_0603_1608Metric_Pad0.98x0.95mm_HandSolder")
+    )
+  )

Commit message: Update label
Parts:
- R3: value 10k -> 150
Changed lines of the file:
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@@
     (in_bom yes) (on_board yes)
     (property "Reference" "R3" (id 0) (at 138.43 91.44 90))
-    (property "Value" "10k" (id 1) (at 138.43 88.9 90))
+    (property "Value" "150" (id 1) (at 138.43 88.9 90))
     (property "Footprint" "Resistor_SMD:R_0603_1608Metric_Pad0.98x0.95mm_HandSolder" (id 2) (at 138.43 89.662 90)
       (effects (font (size 1.27 1.27)) hide)
@@
     )
     (path "/6c5fe62b-2a83-4a65-b6bc-95eae718d02c"
-      (reference "R3") (unit 1) (value "10k") (footprint "Resistor_SMD:R_0603_1608Metric_Pad0.98x0.95mm_HandSolder")
-    )
-  )
+      (reference "R3") (unit 1) (value "150") (footprint "Resistor_SMD:R_0603_1608Metric_Pad0.98x0.95mm_HandSolder")
+    )
+  )
